Commit message: fixed link

File: robots/hand.urdf.xacro (robot description, xacro)
@@ -3,6 +3,6 @@
   <xacro:include filename="$(find barrett_model)/models/hand_top.urdf.xacro"/>
   <!-- Root link is in the world frame-->
-  <link name="world"/>
+  <link name="camera_link"/>
   <!-- BHand -->
-  <xacro:bhand prefix="bhand" parent_link="world" xyz="0.0 0.0 1" rpy="0 0 0"/>
+  <xacro:bhand prefix="bhand" parent_link="camera_link" xyz="0.0 0.0 1" rpy="0 0 0"/>
 </robot>
